File: PCBs/FEHMotorShield/FEHMotorShield.kicad_sch (KiCad schematic)
At the start: 17 parts, among them J1 Conn_01x08_Socket, J10 CONN_03JST-PTH, J11 CONN_03JST-PTH, J12 CONN_03JST-PTH, J13 CONN_03JST-PTH, J2 Conn_01x08_Socket, J3 Conn_01x08_Socket, J4 Conn_01x08_Socket, J5 JST_2MM_MALE, J6 JST_2MM_MALE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

Commit message: Moved PWM pins and added DC-DC converter
Parts:
- removed U1: TSR_1-24150, Converter_DCDC:Converter_DCDC_TRACO_TSR-1_THT, symbol Regulator_Switching:TSR_1-24150
- added C3: 0.1uF, symbol Device:C_Small
- added C4: 44u, symbol Device:C_Small
- added C5: 10uF, symbol Device:C_Polarized_Small
- added C6: 470uF, symbol Device:C_Polarized_Small
- added L1: 1.8uH, symbol Device:L
- added R1: 220k, symbol Device:R_Small
- added R2: 30k, symbol Device:R_Small
- added U1: TPS564242DRLR, TPS564242DRLR_TEX, symbol 2023-08-09_15-07-36:TPS564242DRLR
Connections:
- net +5VA: now also C4.1, L1.2, R1.2, R2.1, U1.5 (EN)
- net +BATT: now also C3.2, C5.1, C6.1, U1.1 (VIN)
- net GND: now also C3.1, C4.2, C5.2, C6.2, R2.2, U1.3 (GND), U1.4 (AGND)
- net PWMA: now also A1.D3 (D3_INT1); no longer A1.D2 (D2_INT0)
- net PWMB: now also A1.D4; no longer A1.D3 (D3_INT1)
- net PWMC: now also A1.D5; no longer A1.D4
- net PWMD: now also A1.D6; no longer A1.D5
- net SERVO1: now also A1.D7; no longer A1.D6
- net SERVO2: now also A1.D8; no longer A1.D7
- net SERVO3: now also A1.D9; no longer A1.D8
- net SERVO4: now also A1.D10; no longer A1.D9
- new net: L1.1, U1.2 (SW)
- new net: R1.1, U1.6 (FB)
Other:
- note added: "Buck Converter Circuit"
- note removed: "Placeholder Buck Converter"
- moved on the sheet: C1, C2, J5
